File: Schematic/LEDMatrix.sch (EAGLE design)
At the start: 29 parts, among them J1 1-2199298-2, SW1 EG1218

Commit message: Corrected files
Parts:
- removed BT1: BS-7, BS-7 snap:BS-7
- removed FRAME1: FRAME-LETTER, SparkFun-Aesthetics:FRAME-LETTER
- added B1: BS-7, BS-7:BS-7
Connections:
- net GND: now also B1.1; no longer BT1.-
- net N$7: now also B1.2; no longer BT1.+
Changed lines of the file:
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@@
 </classes>
 <parts>
-<part name="FRAME1" library="SparkFun-Aesthetics" deviceset="FRAME-LETTER" device=""/>
 <part name="LED1" library="adafruit" deviceset="LED" device="3MM"/>
 <part name="LED2" library="adafruit" deviceset="LED" device="3MM"/>
@@
 <part name="J1" library="8pinsocket" deviceset="1-2199298-2" device=""/>
 <part name="SW1" library="EG1218" deviceset="EG1218" device=""/>
-<part name="BT1" library="BS-7 snap" deviceset="BS-7" device=""/>
+<part name="B1" library="BS-7" deviceset="BS-7" device=""/>
 </parts>
 <sheets>
@@
 </plain>
 <instances>
-<instance part="FRAME1" gate="G$1" x="0" y="0" smashed="yes"/>
-<instance part="FRAME1" gate="V" x="147.32" y="0" smashed="yes">
-<attribute name="LAST_DATE_TIME" x="160.02" y="1.27" size="2.54" layer="94" font="vector"/>
-<attribute name="SHEET" x="233.68" y="1.27" size="2.54" layer="94" font="vector"/>
-<attribute name="DRAWING_NAME" x="162.814" y="17.78" size="2.7432" layer="94" font="vector"/>
-<attribute name="DESIGNER" x="170.434" y="11.176" size="2.7432" layer="94" font="vector"/>
-<attribute name="REV" x="236.22" y="6.604" size="2.7432" layer="94" font="vector"/>
-</instance>
 <instance part="LED1" gate="G$1" x="66.04" y="132.08" smashed="yes">
 <attribute name="NAME" x="69.596" y="127.508" size="1.778" layer="95" rot="R90"/>
@@
 <attribute name="NAME" x="144.5006" y="112.5728" size="3.4798" layer="95" ratio="10" rot="SR0"/>
 </instance>
-<instance part="BT1" gate="G$1" x="175.26" y="99.06" smashed="yes">
-<attribute name="NAME" x="171.45" y="102.87" size="1.778" layer="95"/>
-<attribute name="VALUE" x="171.45" y="93.98" size="1.778" layer="96"/>
+<instance part="B1" gate="A" x="170.18" y="99.06" smashed="yes">
+<attribute name="NAME" x="167.1066" y="101.1428" size="3.4798" layer="95" ratio="10" rot="SR0"/>
+<attribute name="VALUE" x="166.0398" y="93.5228" size="3.4798" layer="96" ratio="10" rot="SR0"/>
 </instance>
 </instances>
@@
 </segment>
 <segment>
-<pinref part="BT1" gate="G$1" pin="-"/>
-<wire x1="182.88" y1="99.06" x2="187.96" y2="99.06" width="0.1524" layer="91"/>
+<wire x1="180.34" y1="99.06" x2="187.96" y2="99.06" width="0.1524" layer="91"/>
 <label x="187.96" y="99.06" size="1.778" layer="95"/>
+<pinref part="B1" gate="A" pin="1"/>
 </segment>
 </net>
@@
 <segment>
 <pinref part="SW1" gate="A" pin="3"/>
-<wire x1="157.48" y1="99.06" x2="167.64" y2="99.06" width="0.1524" layer="91"/>
-<pinref part="BT1" gate="G$1" pin="+"/>
-</segment>
-</net>
+<wire x1="157.48" y1="99.06" x2="170.18" y2="99.06" width="0.1524" layer="91"/>
+<pinref part="B1" gate="A" pin="2"/>
+</segment>
+</net>
